File: LED_Mounting_PoCs/Front_Mount_SMT_LED_PoCs/Front_Mount_SMT_LED_PoCs.sch (KiCad schematic (older format))
At the start: 332 parts, among them J1 Conn_01x08_Male, J2 Conn_01x08_Male, J3 Conn_01x24_Male, U1 HT16D33A

Commit message: finished
Connections:
- net at D103.2 (A), D119.2 (A), D135.2 (A)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: now also D148.1 (K)
- net at D105.2 (A), D121.2 (A), D137.2 (A)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: now also D184.1 (K)
- net at D107.2 (A), D123.2 (A), D139.2 (A)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: now also D211.1 (K)
- net at D111.2 (A), D127.2 (A), D143.2 (A)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: now also D278.1 (K)
Changed lines of the file:
@@
 	10950 9400 10350 9400
 Connection ~ 10350 9400
-$Comp
-L Device:LED_Small D203
-U 1 1 60F4AB7C
-P 10350 9500
-F 0 "D203" V 10396 9430 50  0000 R CNN
-F 1 "LED_Small" V 10305 9430 50  0000 R CNN
-F 2 "LEDs:LED_0603" V 10350 9500 50  0001 C CNN
-F 3 "~" V 10350 9500 50  0001 C CNN
-	1    10350 9500
-	0    -1   -1   0
-$EndComp
 Wire Wire Line
 	10350 9100 10450 9100
@@
 	7950 10600 7350 10600
 Connection ~ 7350 10600
-$Comp
-L Device:LED_Small D127
-U 1 1 60EC7DDE
-P 7350 10700
-F 0 "D127" V 7396 10630 50  0000 R CNN
-F 1 "LED_Small" V 7305 10630 50  0000 R CNN
-F 2 "LEDs:LED_0603" V 7350 10700 50  0001 C CNN
-F 3 "~" V 7350 10700 50  0001 C CNN
-	1    7350 10700
-	0    -1   -1   0
-$EndComp
 Wire Wire Line
 	7350 10300 7950 10300
@@
 Wire Wire Line
 	13450 7800 13450 7500
-Wire Wire Line
-	13400 8100 13450 8100
 Connection ~ 13450 8100
 Wire Wire Line
@@
 	11050 6900 11050 6600
 Wire Wire Line
-	11000 7200 10950 7200
-Wire Wire Line
 	11050 7500 10950 7500
 Connection ~ 11050 7500
 Wire Wire Line
-	11050 7500 11050 6900
+	11050 7500 11050 7200
 Wire Wire Line
 	11050 7800 10950 7800
@@
 Wire Wire Line
 	9850 8400 9850 8700
-Wire Wire Line
-	9800 8700 9850 8700
 Connection ~ 9850 8700
 Wire Wire Line
@@
 Wire Wire Line
 	8550 7200 8650 7200
-Wire Wire Line
-	8600 7500 8650 7500
 Connection ~ 8650 7500
 Wire Wire Line
@@
 Wire Wire Line
 	3550 6350 3150 6350
+$Comp
+L Device:LED_Small D127
+U 1 1 60EC7DDE
+P 7350 10700
+F 0 "D127" V 7396 10630 50  0000 R CNN
+F 1 "LED_Small" V 7305 10630 50  0000 R CNN
+F 2 "LEDs:LED_0603" V 7350 10700 50  0001 C CNN
+F 3 "~" V 7350 10700 50  0001 C CNN
+	1    7350 10700
+	0    -1   -1   0
+$EndComp
+$Comp
+L Device:LED_Small D203
+U 1 1 60F4AB7C
+P 10350 9500
+F 0 "D203" V 10396 9430 50  0000 R CNN
+F 1 "LED_Small" V 10305 9430 50  0000 R CNN
+F 2 "LEDs:LED_0603" V 10350 9500 50  0001 C CNN
+F 3 "~" V 10350 9500 50  0001 C CNN
+	1    10350 9500
+	0    -1   -1   0
+$EndComp
+Wire Wire Line
+	8550 7500 8650 7500
+Wire Wire Line
+	9750 8700 9850 8700
+Wire Wire Line
+	10950 7200 11050 7200
+Connection ~ 11050 7200
+Wire Wire Line
+	11050 7200 11050 6900
+Wire Wire Line
+	13350 8100 13450 8100
 $EndSCHEMATC
